File: practica2/practica.kicad_sch (KiCad schematic)
At the start: 10 parts, among them Q1 BC549, Q2 BC549

Commit message: 1
Parts:
- Q1, Q2: footprint Package_TO_SOT_THT:TO-92_Inline -> Package_TO_SOT_THT:TO-92_Wide
Changed lines of the file:
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@@
       (effects (font (size 1.27 1.27)) (justify left))
     )
-    (property "Footprint" "Package_TO_SOT_THT:TO-92_Inline" (at 168.91 90.805 0)
+    (property "Footprint" "Package_TO_SOT_THT:TO-92_Wide" (at 168.91 90.805 0)
       (effects (font (size 1.27 1.27) italic) (justify left) hide)
     )
@@
       (effects (font (size 1.27 1.27)) (justify left))
     )
-    (property "Footprint" "Package_TO_SOT_THT:TO-92_Inline" (at 181.61 80.645 0)
+    (property "Footprint" "Package_TO_SOT_THT:TO-92_Wide" (at 181.61 80.645 0)
       (effects (font (size 1.27 1.27) italic) (justify left) hide)
     )

Commit message: 1
Parts:
- removed D1: GL5516, Diode_THT:D_A-405_P10.16mm_Horizontal, symbol Device:D_Photo
- removed D2: 1N4148, Diode_THT:D_A-405_P10.16mm_Horizontal, symbol Device:D
- added D2: LED, LED_THT:LED_D2.0mm_W4.8mm_H2.5mm_FlatTop, symbol Device:LED
- added R4: 33, Resistor_THT:R_Axial_DIN0204_L3.6mm_D1.6mm_P7.62mm_Horizontal, symbol Device:R
- added R5: R_Photo, Resistor_THT:R_Axial_DIN0204_L3.6mm_D1.6mm_P5.08mm_Vertical, symbol Device:R_Photo
Connections:
- net +12V: now also R4.1, R5.1
- net at R1.1, RV1.1, RV1.2: now also R5.2
- net out-: no longer names the net of Q2.1 (C)
- net out-: now also D2.2 (A)
- new net: D2.1 (K), R4.2
Other:
- moved on the sheet: C1, Q2, RV1

Commit message: 1
Parts:
- R1: renamed from R5; value R_Photo -> GL5516
- renumbered RV1 to R2, R1 to R3, R2 to R4, R3 to R5, R4 to R6, D2 to VD2, Q1 to VT1, Q2 to VT2
Connections:
- net at R6.2: now also VD2.2 (A); no longer VD2.1 (K)
- net at VT2.1 (C): now also VD2.1 (K); no longer VD2.2 (A)
Other:
- moved on the sheet: VD2
Changed lines of the file:
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@@
   (symbol (lib_id "Device:R") (at 175.26 63.5 90) (unit 1)
     (in_bom yes) (on_board yes) (dnp no) (fields_autoplaced)
-    (property "Reference" "R4" (at 175.26 58.42 90)
-      (effects (font (size 1.27 1.27)))
-    )
-    (property "Value" "33" (at 175.26 60.96 90)
+    (property "Reference" "R6" (at 175.26 57.15 90)
+      (effects (font (size 1.27 1.27)))
+    )
+    (property "Value" "33" (at 175.26 59.69 90)
       (effects (font (size 1.27 1.27)))
     )
@@
       (project "practica"
         (path "/c2584096-a91d-4080-a75c-dc164545fb5d"
-          (reference "R4") (unit 1)
+          (reference "R6") (unit 1)
         )
       )
@@
   (symbol (lib_id "Device:R_Photo") (at 138.43 76.2 0) (unit 1)
     (in_bom yes) (on_board yes) (dnp no)
-    (property "Reference" "R5" (at 140.97 74.93 0)
-      (effects (font (size 1.27 1.27)) (justify left))
-    )
-    (property "Value" "R_Photo" (at 140.97 77.47 0)
+    (property "Reference" "R1" (at 140.97 74.93 0)
+      (effects (font (size 1.27 1.27)) (justify left))
+    )
+    (property "Value" "GL5516" (at 140.97 77.47 0)
       (effects (font (size 1.27 1.27)) (justify left))
     )
@@
       (project "practica"
         (path "/c2584096-a91d-4080-a75c-dc164545fb5d"
-          (reference "R5") (unit 1)
+          (reference "R1") (unit 1)
         )
       )
@@
   (symbol (lib_id "Device:R_Potentiometer") (at 138.43 99.06 0) (unit 1)
     (in_bom yes) (on_board yes) (dnp no) (fields_autoplaced)
-    (property "Reference" "RV1" (at 135.89 97.7899 0)
+    (property "Reference" "R2" (at 135.89 97.79 0)
       (effects (font (size 1.27 1.27)) (justify right))
     )
-    (property "Value" "10k" (at 135.89 100.3299 0)
+    (property "Value" "10k" (at 135.89 100.33 0)
       (effects (font (size 1.27 1.27)) (justify right))
     )
@@
       (project "practica"
         (path "/c2584096-a91d-4080-a75c-dc164545fb5d"
-          (reference "RV1") (unit 1)
+          (reference "R2") (unit 1)
         )
       )
@@
   (symbol (lib_id "Transistor_BJT:BC549") (at 163.83 88.9 0) (unit 1)
     (in_bom yes) (on_board yes) (dnp no) (fields_autoplaced)
-    (property "Reference" "Q1" (at 168.91 87.6299 0)
-      (effects (font (size 1.27 1.27)) (justify left))
-    )
-    (property "Value" "BC549" (at 168.91 90.1699 0)
+    (property "Reference" "VT1" (at 168.91 87.63 0)
+      (effects (font (size 1.27 1.27)) (justify left))
+    )
+    (property "Value" "BC549" (at 168.91 90.17 0)
       (effects (font (size 1.27 1.27)) (justify left))
     )
@@
       (project "practica"
         (path "/c2584096-a91d-4080-a75c-dc164545fb5d"
-          (reference "Q1") (unit 1)
+          (reference "VT1") (unit 1)
         )
       )
@@
   (symbol (lib_id "Device:R") (at 166.37 101.6 0) (unit 1)
     (in_bom yes) (on_board yes) (dnp no) (fields_autoplaced)
-    (property "Reference" "R3" (at 168.91 100.3299 0)
-      (effects (font (size 1.27 1.27)) (justify left))
-    )
-    (property "Value" "33" (at 168.91 102.8699 0)
+    (property "Reference" "R5" (at 168.91 100.33 0)
+      (effects (font (size 1.27 1.27)) (justify left))
+    )
+    (property "Value" "33" (at 168.91 102.87 0)
       (effects (font (size 1.27 1.27)) (justify left))
     )
@@
       (project "practica"
         (path "/c2584096-a91d-4080-a75c-dc164545fb5d"
-          (reference "R3") (unit 1)
+          (reference "R5") (unit 1)
         )
       )
@@
   (symbol (lib_id "Device:R") (at 166.37 71.12 0) (unit 1)
     (in_bom yes) (on_board yes) (dnp no) (fields_autoplaced)
-    (property "Reference" "R2" (at 168.91 69.8499 0)
-      (effects (font (size 1.27 1.27)) (justify left))
-    )
-    (property "Value" "3,3k" (at 168.91 72.3899 0)
+    (property "Reference" "R4" (at 168.91 69.85 0)
+      (effects (font (size 1.27 1.27)) (justify left))
+    )
+    (property "Value" "3,3k" (at 168.91 72.39 0)
       (effects (font (size 1.27 1.27)) (justify left))
     )
@@
       (project "practica"
         (path "/c2584096-a91d-4080-a75c-dc164545fb5d"
-          (reference "R2") (unit 1)
+          (reference "R4") (unit 1)
         )
       )
@@
   (symbol (lib_id "Device:R") (at 147.32 88.9 90) (unit 1)
     (in_bom yes) (on_board yes) (dnp no) (fields_autoplaced)
-    (property "Reference" "R1" (at 147.32 82.55 90)
+    (property "Reference" "R3" (at 147.32 82.55 90)
       (effects (font (size 1.27 1.27)))
     )
@@
       (project "practica"
         (path "/c2584096-a91d-4080-a75c-dc164545fb5d"
-          (reference "R1") (unit 1)
+          (reference "R3") (unit 1)
         )
       )
@@
   (symbol (lib_id "Transistor_BJT:BC549") (at 180.34 78.74 0) (unit 1)
     (in_bom yes) (on_board yes) (dnp no) (fields_autoplaced)
-    (property "Reference" "Q2" (at 185.42 77.4699 0)
-      (effects (font (size 1.27 1.27)) (justify left))
-    )
-    (property "Value" "BC549" (at 185.42 80.0099 0)
+    (property "Reference" "VT2" (at 185.42 77.47 0)
+      (effects (font (size 1.27 1.27)) (justify left))
+    )
+    (property "Value" "BC549" (at 185.42 80.01 0)
       (effects (font (size 1.27 1.27)) (justify left))
     )
@@
       (project "practica"
         (path "/c2584096-a91d-4080-a75c-dc164545fb5d"
-          (reference "Q2") (unit 1)
-        )
-      )
-    )
-  )
-  (symbol (lib_id "Device:LED") (at 182.88 68.58 90) (mirror x) (unit 1)
+          (reference "VT2") (unit 1)
+        )
+      )
+    )
+  )
+  (symbol (lib_id "Device:LED") (at 182.88 68.58 90) (unit 1)
     (in_bom yes) (on_board yes) (dnp no)
-    (property "Reference" "D2" (at 187.96 67.31 90)
-      (effects (font (size 1.27 1.27)) (justify left))
-    )
-    (property "Value" "LED" (at 189.23 69.85 90)
+    (property "Reference" "VD2" (at 187.96 69.85 90)
+      (effects (font (size 1.27 1.27)) (justify left))
+    )
+    (property "Value" "LED" (at 189.23 67.31 90)
       (effects (font (size 1.27 1.27)) (justify left))
     )
@@
       (project "practica"
         (path "/c2584096-a91d-4080-a75c-dc164545fb5d"
-          (reference "D2") (unit 1)
-        )
-      )
+          (reference "VD2") (unit 1)
+        )
+      )
